File: PCB/PiicoDev-Colour-Sensor-VEML6040.kicad_pcb (KiCad board)
At the start: 2 copper layers, 25.4 x 25.4 mm, 23 parts, among them J1 , J2 , J3 Conn_PiicoDev_header_01x04_Ma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, J4 Conn_01x01_Male, Q1 BSS138, U1 VEML6040

Commit message: Change 4k7 resistors to 10k
Parts:
- R2, R5: value 4.7k -> 10k
- R3, R4: value 4k7 -> 10k
